File: pcb/body/_autosave-pickuppair.kicad_sch (KiCad schematic)
At the start: 26 parts, among them U2 TL072

Commit message: initial layout
Parts:
- renumbered R14 to R10, R13 to R9, RV2 to RV3, RV5 to RV4
