File: pcb/body/body.kicad_sch (KiCad schematic)
At the start: 27 parts, among them J1 FRETBOARD_CONNECTION, J2 BRIDGE_GROUND, J3 Conn_01x08_Socket, J4 AudioJack3_SwitchTR, J5 External_connections, J6 OUTPUTS_234, U1 Teensy4.1

Commit message: getting there
Connections:
- net +3.3V: now also J1.1 (Pin_1), U1.15 (3V3), U1.46 (3V3)
- net GND: now also J1.2 (Pin_2), U1.1 (GND), U1.34 (GND), U1.47 (GND)
- net FRET_CLOCK: now reaches J1.3 (Pin_3)
- net FRET_CLOCK: now also U1.21 (29_TX7)
- net FRET_LOAD: now reaches J1.4 (Pin_4)
- net FRET_LOAD: now also U1.22 (30_CRX3)
- net FRET_DATA: now reaches J1.5 (Pin_5)
- net FRET_DATA: now also U1.23 (31_CTX3)
- net +5V: now reaches U1.48 (VIN)
- no-connect marks 11 -> 39

Commit message: not much
Parts:
- J1: footprint Connector_PinHeader_2.54mm:PinHeader_1x05_P2.54mm_Horizontal -> bjarkarbody:jst zh fretboard connector; symbol Connector:Conn_01x05_Pin -> Connector:Conn_01x06_Pin
- J3: value Conn_01x08_Socket -> GK3_socket
Connections:
- no-connect marks 39 -> 40
Other:
- note added: "S8B-ZR, pitch 1.5mm"
- note removed: "B8B-ZR, pitch 1.5mm"
Changed lines of the file:
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@@
   (no_connect (at 86.36 156.21))
   (no_connect (at 201.93 106.68))
+  (no_connect (at 33.02 78.74))
   (no_connect (at 86.36 143.51))
   (no_connect (at 30.48 133.35))
@@
     (effects (font (size 1.27 1.27)) (justify left bottom))
   )
-  (text "B8B-ZR, pitch 1.5mm" (at 76.2 24.13 0)
+  (text "S8B-ZR, pitch 1.5mm" (at 76.2 24.13 0)
     (effects (font (size 1.27 1.27)) (justify left bottom))
   )
@@
     )
   )
-  (symbol (lib_id "Connector:Conn_01x05_Pin") (at 27.94 71.12 0) (unit 1)
+  (symbol (lib_id "Connector:Conn_01x06_Pin") (at 27.94 71.12 0) (unit 1)
     (in_bom yes) (on_board yes) (dnp no) (fields_autoplaced)
     (property "Reference" "J1" (at 28.575 62.9539 0)
@@
       (effects (font (size 1.27 1.27)))
     )
-    (property "Footprint" "Connector_PinHeader_2.54mm:PinHeader_1x05_P2.54mm_Horizontal" (at 27.94 71.12 0)
+    (property "Footprint" "bjarkarbody:jst zh fretboard connector" (at 27.94 71.12 0)
       (effects (font (size 1.27 1.27)) hide)
     )
@@
     (pin "4")
     (pin "5")
+    (pin "6")
     (instances
       (project "body"
@@
       (effects (font (size 1.27 1.27)) (justify left))
     )
-    (property "Value" "Conn_01x08_Socket" (at 83.1088 38.1073 0)
+    (property "Value" "GK3_socket" (at 83.1088 38.1073 0)
       (effects (font (size 1.27 1.27)) (justify left))
     )

Commit message: body pcb zero errors
Parts:
- added PB1, PB10, PB100, PB101, PB102, PB103, PB104, PB105, PB106, PB107, PB108, PB109, PB11, PB110, PB111, PB112, PB113, PB114, PB115, PB116, PB117, PB118, PB119, PB12, PB120, PB121, PB122, PB123, PB124, PB125, PB126, PB127, PB128, PB129, PB13, PB130, PB131, PB132, PB133, PB134, PB135, PB136, PB137, PB138, PB139, PB14, PB140, PB141, PB142, PB143, PB144, PB15, PB16, PB17, PB18, PB19, PB2, PB20, PB21, PB22, PB23, PB24, PB25, PB26, PB27, PB28, PB29, PB3, PB30, PB31, PB32, PB33, PB34, PB35, PB36, PB37, PB38, PB39, PB4, PB40, PB41, PB42, PB43, PB44, PB45, PB46, PB47, PB48, PB49, PB5, PB50, PB51, PB52, PB53, PB54, PB55, PB56, PB57, PB58, PB59, PB6, PB60, PB61, PB62, PB63, PB64, PB65, PB66, PB67, PB68, PB69, PB7, PB70, PB71, PB72, PB73, PB74, PB75, PB76, PB77, PB78, PB79, PB8, PB80, PB81, PB82, PB83, PB84, PB85, PB86, PB87, PB88, PB89, PB9, PB90, PB91, PB92, PB93, PB94, PB95, PB96, PB97, PB98, PB99: perfboard_pin, bjarkarbody:perfboard pin, symbol bjarkarbody:perfboard_pin
- J3: footprint Connector_Wuerth:Wuerth_WR-WTB_64800811622_1x08_P1.50mm_Vertical -> bjarkarbody:gk3 connector THT
