File: pcb/body/pickuppair.kicad_sch (KiCad schematic)
At the start: 26 parts, among them U2 TL072

Commit message: lots more layout
Parts:
- RV3: renamed from RV2; footprint Potentiometer_THT:Potentiometer_Bourns_3296W_Vertical -> Potentiometer_THT:Potentiometer_Bourns_3296P_Horizontal
- RV4: renamed from RV5; footprint Potentiometer_THT:Potentiometer_Bourns_3296W_Vertical -> Potentiometer_THT:Potentiometer_Bourns_3296P_Horizontal
- renumbered C6 to C10, C7 to C11, C8 to C12, C9 to C13, C10 to C14, C11 to C15, C1 to C5, C2 to C6, C3 to C7, C4 to C8, C5 to C9, R1 to R13, R2 to R14, R3 to R15, R4 to R16, R5 to R17, R6 to R18, R7 to R19, R8 to R20, R13 to R21, R14 to R22
Connections:
- no-connect marks 1 -> 2
