File: pcb/body/codec.kicad_sch (KiCad schematic)
At the start: 9 parts, among them U5 SGTL5000XNLA3

Commit message: getting there
Changed lines of the file:
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@@
   (junction (at 139.7 66.04) (diameter 0) (color 0 0 0 0)
   )
+  (junction (at 154.94 68.58) (diameter 0) (color 0 0 0 0)
+  )
   (junction (at 115.57 73.66) (diameter 0) (color 0 0 0 0)
   )
@@
     (stroke (width 0) (type default))
   )
-  (wire (pts (xy 154.94 53.34) (xy 154.94 72.39))
+  (wire (pts (xy 154.94 53.34) (xy 154.94 68.58))
     (stroke (width 0) (type default))
   )
@@
   )
   (wire (pts (xy 139.7 66.04) (xy 149.86 66.04))
+    (stroke (width 0) (type default))
+  )
+  (wire (pts (xy 154.94 68.58) (xy 154.94 72.39))
     (stroke (width 0) (type default))
   )
@@
         )
       )
+    )
+  )
+  (symbol (lib_id "power:PWR_FLAG") (at 154.94 68.58 270) (unit 1)
+    (in_bom yes) (on_board yes) (dnp no) (fields_autoplaced)
+    (property "Reference" "#FLG01" (at 156.845 68.58 0)
+      (effects (font (size 1.27 1.27)) hide)
+    )
+    (property "Value" "PWR_FLAG" (at 158.115 68.8968 90)
+      (effects (font (size 1.27 1.27)) (justify left))
+    )
+    (property "Footprint" "" (at 154.94 68.58 0)
+      (effects (font (size 1.27 1.27)) hide)
+    )
+    (property "Datasheet" "~" (at 154.94 68.58 0)
+      (effects (font (size 1.27 1.27)) hide)
+    )
+    (pin "1")
+    (instances
+      (project "body"
+        (path "/392bd065-a607-4eff-83a3-798a3e7c56fd/1a6ed37c-c9ef-40ab-9127-b7ac3319730a"
+          (reference "#FLG01") (unit 1)
+        )
+        (path "/392bd065-a607-4eff-83a3-798a3e7c56fd/0ec532ff-7996-4c16-be23-c6d234e49048"
+          (reference "#FLG03") (unit 1)
+        )
+        (path "/392bd065-a607-4eff-83a3-798a3e7c56fd/2085223b-db3d-43d9-b30b-97ab8cd1e664"
+          (reference "#FLG04") (unit 1)
+        )
+        (path "/392bd065-a607-4eff-83a3-798a3e7c56fd/28e071a9-d765-4c5b-8e6e-bd238b4a8a54"
+          (reference "#FLG05") (unit 1)
+        )
+      )
