File: pcb/body/body.kicad_pcb (KiCad board)
At the start: 4 copper layers, 90 x 120 mm, 149 parts, among them J1 FRETBOARD_CONNECTION, J2 BRIDGE_GROUND, J3 Conn_01x08_Socket, J4 AudioJack3_SwitchTR, J5 External_connections, J6 OUTPUTS_234, J7 Battery_Power, U1 Teensy4.1, U2 TL072, U3 TL072, U4 TL072, U5 SGTL5000XNLA3, U6 SGTL5000XNLA3, U7 SGTL5000XNLA3, U8 TPS54331DR, U9 AP7313-18SAG

Commit message: getting there
Connections:
- J1 pad 1: unconnected-(J1-Pin_1-Pad1) -> +3.3V
- J1 pad 2: unconnected-(J1-Pin_2-Pad2) -> GND
- J1 pad 3: unconnected-(J1-Pin_3-Pad3) -> FRET_CLOCK
- J1 pad 4: unconnected-(J1-Pin_4-Pad4) -> FRET_LOAD
- J1 pad 5: unconnected-(J1-Pin_5-Pad5) -> FRET_DATA
- U1 pad 1: unconnected-(U1-GND-Pad1) -> GND
- U1 pad 15: unconnected-(U1-3V3-Pad15) -> +3.3V
- U1 pad 21: unconnected-(U1-29_TX7-Pad21) -> FRET_CLOCK
- U1 pad 22: unconnected-(U1-30_CRX3-Pad22) -> FRET_LOAD
- U1 pad 23: unconnected-(U1-31_CTX3-Pad23) -> FRET_DATA
- U1 pad 34: unconnected-(U1-GND-Pad34) -> GND
- U1 pad 46: unconnected-(U1-3V3-Pad46) -> +3.3V
- U1 pad 47: unconnected-(U1-GND-Pad47) -> GND
- U1 pad 48: unconnected-(U1-VIN-Pad48) -> +5V
Routing:
- net FRET_CLOCK: track 0.00 -> 28.7 mm
- net FRET_LOAD: track 0.00 -> 26.8 mm
- net +5V: track 5.91 -> 31.2 mm
- net FRET_DATA: track 0.00 -> 24.9 mm
- net +3.3V: track 61.0 -> 80.6 mm
- net GND: track 163.5 -> 171.1 mm
- net unconnected-(U1-VIN-Pad48): track 2.54 -> 0.00 mm
- net unconnected-(U1-GND-Pad47): track 2.54 -> 0.00 mm
- net unconnected-(U1-GND-Pad34): track 2.54 -> 0.00 mm
- net unconnected-(U1-GND-Pad1): track 2.54 -> 0.00 mm
- net unconnected-(U1-3V3-Pad46): track 2.54 -> 0.00 mm
- net unconnected-(U1-3V3-Pad15): track 2.54 -> 0.00 mm
- net unconnected-(U1-31_CTX3-Pad23): track 2.54 -> 0.00 mm
- net unconnected-(U1-30_CRX3-Pad22): track 2.54 -> 0.00 mm
- net unconnected-(U1-29_TX7-Pad21): track 2.54 -> 0.00 mm
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
Commit message: not much
Parts:
- J1: footprint Connector_PinHeader_2.54mm:PinHeader_1x05_P2.54mm_Horizontal -> bjarkarbody:jst zh fretboard connector; moved to F.Cu
- moved J1 7.28 mm to (147.0, 42.0), turned to 180 degrees
Routing:
- net unconnected-(J1-Pin_6-Pad6): track 0.00 -> 10.0 mm
- net FRET_CLOCK: track 28.7 -> 37.1 mm
- net +3.3V: track 80.6 -> 72.3 mm, vias 15 -> 16
- net FRET_LOAD: track 26.8 -> 31.1 mm
- net GND: track 171.1 -> 175.1 mm, vias 52 -> 53
- net FRET_DATA: track 24.9 -> 23.8 mm

Commit message: body pcb zero errors
Parts:
- added PB1: perfboard_pin, bjarkarbody:perfboard pin, F.Cu at (173.3, 60.8)
- added PB10: perfboard_pin, bjarkarbody:perfboard pin, F.Cu at (173.3, 83.7)
- added PB100: perfboard_pin, bjarkarbody:perfboard pin, F.Cu at (178.4, 98.9)
- added PB101: perfboard_pin, bjarkarbody:perfboard pin, F.Cu at (178.4, 101.4)
- added PB102: perfboard_pin, bjarkarbody:perfboard pin, F.Cu at (178.4, 104.0)
- added PB103: perfboard_pin, bjarkarbody:perfboard pin, F.Cu at (178.4, 106.5)
- added PB104: perfboard_pin, bjarkarbody:perfboard pin, F.Cu at (178.4, 109.1)
- added PB105: perfboard_pin, bjarkarbody:perfboard pin, F.Cu at (178.4, 111.6)
- added PB106: perfboard_pin, bjarkarbody:perfboard pin, F.Cu at (178.4, 114.1)
- added PB107: perfboard_pin, bjarkarbody:perfboard pin, F.Cu at (178.4, 116.7)
- added PB108: perfboard_pin, bjarkarbody:perfboard pin, F.Cu at (178.4, 119.2)
- added PB109: perfboard_pin, bjarkarbody:perfboard pin, F.Cu at (181.0, 91.3)
- added PB11: perfboard_pin, bjarkarbody:perfboard pin, F.Cu at (173.3, 86.2)
- added PB110: perfboard_pin, bjarkarbody:perfboard pin, F.Cu at (181.0, 93.8)
- added PB111: perfboard_pin, bjarkarbody:perfboard pin, F.Cu at (181.0, 96.4)
- added PB112: perfboard_pin, bjarkarbody:perfboard pin, F.Cu at (181.0, 98.9)
- added PB113: perfboard_pin, bjarkarbody:perfboard pin, F.Cu at (181.0, 101.4)
- added PB114: perfboard_pin, bjarkarbody:perfboard pin, F.Cu at (181.0, 104.0)
- added PB115: perfboard_pin, bjarkarbody:perfboard pin, F.Cu at (181.0, 106.5)
- added PB116: perfboard_pin, bjarkarbody:perfboard pin, F.Cu at (181.0, 109.1)
- added PB117: perfboard_pin, bjarkarbody:perfboard pin, F.Cu at (181.0, 111.6)
- added PB118: perfboard_pin, bjarkarbody:perfboard pin, F.Cu at (181.0, 114.1)
- added PB119: perfboard_pin, bjarkarbody:perfboard pin, F.Cu at (181.0, 116.7)
- added PB12: perfboard_pin, bjarkarbody:perfboard pin, F.Cu at (173.3, 88.7)
- added PB120: perfboard_pin, bjarkarbody:perfboard pin, F.Cu at (181.0, 119.2)
- added PB121: perfboard_pin, bjarkarbody:perfboard pin, F.Cu at (183.5, 91.3)
- added PB122: perfboard_pin, bjarkarbody:perfboard pin, F.Cu at (183.5, 93.8)
- added PB123: perfboard_pin, bjarkarbody:perfboard pin, F.Cu at (183.5, 96.4)
- added PB124: perfboard_pin, bjarkarbody:perfboard pin, F.Cu at (183.5, 98.9)
- added PB125: perfboard_pin, bjarkarbody:perfboard pin, F.Cu at (183.5, 101.4)
- added PB126: perfboard_pin, bjarkarbody:perfboard pin, F.Cu at (183.5, 104.0)
- added PB127: perfboard_pin, bjarkarbody:perfboard pin, F.Cu at (183.5, 106.5)
- added PB128: perfboard_pin, bjarkarbody:perfboard pin, F.Cu at (183.5, 109.1)
- added PB129: perfboard_pin, bjarkarbody:perfboard pin, F.Cu at (183.5, 111.6)
- added PB13: perfboard_pin, bjarkarbody:perfboard pin, F.Cu at (175.9, 60.8)
- added PB130: perfboard_pin, bjarkarbody:perfboard pin, F.Cu at (183.5, 114.1)
- added PB131: perfboard_pin, bjarkarbody:perfboard pin, F.Cu at (183.5, 116.7)
- added PB132: perfboard_pin, bjarkarbody:perfboard pin, F.Cu at (183.5, 119.2)
- added PB133: perfboard_pin, bjarkarbody:perfboard pin, F.Cu at (186.1, 91.3)
- added PB134: perfboard_pin, bjarkarbody:perfboard pin, F.Cu at (186.1, 93.8)
- added PB135: perfboard_pin, bjarkarbody:perfboard pin, F.Cu at (186.1, 96.4)
- added PB136: perfboard_pin, bjarkarbody:perfboard pin, F.Cu at (186.1, 98.9)
- added PB137: perfboard_pin, bjarkarbody:perfboard pin, F.Cu at (186.1, 101.4)
- added PB138: perfboard_pin, bjarkarbody:perfboard pin, F.Cu at (186.1, 104.0)
- added PB139: perfboard_pin, bjarkarbody:perfboard pin, F.Cu at (186.1, 106.5)
- added PB14: perfboard_pin, bjarkarbody:perfboard pin, F.Cu at (175.9, 63.3)
- added PB140: perfboard_pin, bjarkarbody:perfboard pin, F.Cu at (186.1, 109.1)
- added PB141: perfboard_pin, bjarkarbody:perfboard pin, F.Cu at (186.1, 111.6)
- added PB142: perfboard_pin, bjarkarbody:perfboard pin, F.Cu at (186.1, 114.1)
- added PB143: perfboard_pin, bjarkarbody:perfboard pin, F.Cu at (186.1, 116.7)
- added PB144: perfboard_pin, bjarkarbody:perfboard pin, F.Cu at (186.1, 119.2)
- added PB15: perfboard_pin, bjarkarbody:perfboard pin, F.Cu at (175.9, 65.9)
- added PB16: perfboard_pin, bjarkarbody:perfboard pin, F.Cu at (175.9, 68.4)
- added PB17: perfboard_pin, bjarkarbody:perfboard pin, F.Cu at (175.9, 71.0)
- added PB18: perfboard_pin, bjarkarbody:perfboard pin, F.Cu at (175.9, 73.5)
- added PB19: perfboard_pin, bjarkarbody:perfboard pin, F.Cu at (175.9, 76.0)
- added PB2: perfboard_pin, bjarkarbody:perfboard pin, F.Cu at (173.3, 63.3)
- added PB20: perfboard_pin, bjarkarbody:perfboard pin, F.Cu at (175.9, 78.6)
- added PB21: perfboard_pin, bjarkarbody:perfboard pin, F.Cu at (175.9, 81.1)
- added PB22: perfboard_pin, bjarkarbody:perfboard pin, F.Cu at (175.9, 83.7)
- added PB23: perfboard_pin, bjarkarbody:perfboard pin, F.Cu at (175.9, 86.2)
- added PB24: perfboard_pin, bjarkarbody:perfboard pin, F.Cu at (175.9, 88.7)
- added PB25: perfboard_pin, bjarkarbody:perfboard pin, F.Cu at (178.4, 60.8)
- added PB26: perfboard_pin, bjarkarbody:perfboard pin, F.Cu at (178.4, 63.3)
- added PB27: perfboard_pin, bjarkarbody:perfboard pin, F.Cu at (178.4, 65.9)
- added PB28: perfboard_pin, bjarkarbody:perfboard pin, F.Cu at (178.4, 68.4)
- added PB29: perfboard_pin, bjarkarbody:perfboard pin, F.Cu at (178.4, 71.0)
- added PB3: perfboard_pin, bjarkarbody:perfboard pin, F.Cu at (173.3, 65.9)
- added PB30: perfboard_pin, bjarkarbody:perfboard pin, F.Cu at (178.4, 73.5)
- added PB31: perfboard_pin, bjarkarbody:perfboard pin, F.Cu at (178.4, 76.0)
- added PB32: perfboard_pin, bjarkarbody:perfboard pin, F.Cu at (178.4, 78.6)
- added PB33: perfboard_pin, bjarkarbody:perfboard pin, F.Cu at (178.4, 81.1)
- added PB34: perfboard_pin, bjarkarbody:perfboard pin, F.Cu at (178.4, 83.7)
- added PB35: perfboard_pin, bjarkarbody:perfboard pin, F.Cu at (178.4, 86.2)
- added PB36: perfboard_pin, bjarkarbody:perfboard pin, F.Cu at (178.4, 88.7)
- added PB37: perfboard_pin, bjarkarbody:perfboard pin, F.Cu at (181.0, 60.8)
- added PB38: perfboard_pin, bjarkarbody:perfboard pin, F.Cu at (181.0, 63.3)
- added PB39: perfboard_pin, bjarkarbody:perfboard pin, F.Cu at (181.0, 65.9)
- added PB4: perfboard_pin, bjarkarbody:perfboard pin, F.Cu at (173.3, 68.4)
- added PB40: perfboard_pin, bjarkarbody:perfboard pin, F.Cu at (181.0, 68.4)
- added PB41: perfboard_pin, bjarkarbody:perfboard pin, F.Cu at (181.0, 71.0)
- added PB42: perfboard_pin, bjarkarbody:perfboard pin, F.Cu at (181.0, 73.5)
- added PB43: perfboard_pin, bjarkarbody:perfboard pin, F.Cu at (181.0, 76.0)
- added PB44: perfboard_pin, bjarkarbody:perfboard pin, F.Cu at (181.0, 78.6)
- added PB45: perfboard_pin, bjarkarbody:perfboard pin, F.Cu at (181.0, 81.1)
- added PB46: perfboard_pin, bjarkarbody:perfboard pin, F.Cu at (181.0, 83.7)
- added PB47: perfboard_pin, bjarkarbody:perfboard pin, F.Cu at (181.0, 86.2)
- added PB48: perfboard_pin, bjarkarbody:perfboard pin, F.Cu at (181.0, 88.7)
- added PB49: perfboard_pin, bjarkarbody:perfboard pin, F.Cu at (183.5, 60.8)
- added PB5: perfboard_pin, bjarkarbody:perfboard pin, F.Cu at (173.3, 71.0)
- added PB50: perfboard_pin, bjarkarbody:perfboard pin, F.Cu at (183.5, 63.3)
- added PB51: perfboard_pin, bjarkarbody:perfboard pin, F.Cu at (183.5, 65.9)
- added PB52: perfboard_pin, bjarkarbody:perfboard pin, F.Cu at (183.5, 68.4)
- added PB53: perfboard_pin, bjarkarbody:perfboard pin, F.Cu at (183.5, 71.0)
- added PB54: perfboard_pin, bjarkarbody:perfboard pin, F.Cu at (183.5, 73.5)
- added PB55: perfboard_pin, bjarkarbody:perfboard pin, F.Cu at (183.5, 76.0)
- added PB56: perfboard_pin, bjarkarbody:perfboard pin, F.Cu at (183.5, 78.6)
- added PB57: perfboard_pin, bjarkarbody:perfboard pin, F.Cu at (183.5, 81.1)
- added PB58: perfboard_pin, bjarkarbody:perfboard pin, F.Cu at (183.5, 83.7)
- added PB59: perfboard_pin, bjarkarbody:perfboard pin, F.Cu at (183.5, 86.2)
- added PB6: perfboard_pin, bjarkarbody:perfboard pin, F.Cu at (173.3, 73.5)
- added PB60: perfboard_pin, bjarkarbody:perfboard pin, F.Cu at (183.5, 88.7)
- added PB61: perfboard_pin, bjarkarbody:perfboard pin, F.Cu at (186.1, 60.8)
- added PB62: perfboard_pin, bjarkarbody:perfboard pin, F.Cu at (186.1, 63.3)
- added PB63: perfboard_pin, bjarkarbody:perfboard pin, F.Cu at (186.1, 65.9)
- added PB64: perfboard_pin, bjarkarbody:perfboard pin, F.Cu at (186.1, 68.4)
- added PB65: perfboard_pin, bjarkarbody:perfboard pin, F.Cu at (186.1, 71.0)
- added PB66: perfboard_pin, bjarkarbody:perfboard pin, F.Cu at (186.1, 73.5)
- added PB67: perfboard_pin, bjarkarbody:perfboard pin, F.Cu at (186.1, 76.0)
- added PB68: perfboard_pin, bjarkarbody:perfboard pin, F.Cu at (186.1, 78.6)
- added PB69: perfboard_pin, bjarkarbody:perfboard pin, F.Cu at (186.1, 81.1)
- added PB7: perfboard_pin, bjarkarbody:perfboard pin, F.Cu at (173.3, 76.0)
- added PB70: perfboard_pin, bjarkarbody:perfboard pin, F.Cu at (186.1, 83.7)
- added PB71: perfboard_pin, bjarkarbody:perfboard pin, F.Cu at (186.1, 86.2)
- added PB72: perfboard_pin, bjarkarbody:perfboard pin, F.Cu at (186.1, 88.7)
- added PB73: perfboard_pin, bjarkarbody:perfboard pin, F.Cu at (173.3, 91.3)
- added PB74: perfboard_pin, bjarkarbody:perfboard pin, F.Cu at (173.3, 93.8)
- added PB75: perfboard_pin, bjarkarbody:perfboard pin, F.Cu at (173.3, 96.4)
- added PB76: perfboard_pin, bjarkarbody:perfboard pin, F.Cu at (173.3, 98.9)
- added PB77: perfboard_pin, bjarkarbody:perfboard pin, F.Cu at (173.3, 101.4)
- added PB78: perfboard_pin, bjarkarbody:perfboard pin, F.Cu at (173.3, 104.0)
- added PB79: perfboard_pin, bjarkarbody:perfboard pin, F.Cu at (173.3, 106.5)
- added PB8: perfboard_pin, bjarkarbody:perfboard pin, F.Cu at (173.3, 78.6)
- added PB80: perfboard_pin, bjarkarbody:perfboard pin, F.Cu at (173.3, 109.1)
- added PB81: perfboard_pin, bjarkarbody:perfboard pin, F.Cu at (173.3, 111.6)
- added PB82: perfboard_pin, bjarkarbody:perfboard pin, F.Cu at (173.3, 114.1)
- added PB83: perfboard_pin, bjarkarbody:perfboard pin, F.Cu at (173.3, 116.7)
- added PB84: perfboard_pin, bjarkarbody:perfboard pin, F.Cu at (173.3, 119.2)
- added PB85: perfboard_pin, bjarkarbody:perfboard pin, F.Cu at (175.9, 91.3)
- added PB86: perfboard_pin, bjarkarbody:perfboard pin, F.Cu at (175.9, 93.8)
- added PB87: perfboard_pin, bjarkarbody:perfboard pin, F.Cu at (175.9, 96.4)
- added PB88: perfboard_pin, bjarkarbody:perfboard pin, F.Cu at (175.9, 98.9)
- added PB89: perfboard_pin, bjarkarbody:perfboard pin, F.Cu at (175.9, 101.4)
- added PB9: perfboard_pin, bjarkarbody:perfboard pin, F.Cu at (173.3, 81.1)
- added PB90: perfboard_pin, bjarkarbody:perfboard pin, F.Cu at (175.9, 104.0)
- added PB91: perfboard_pin, bjarkarbody:perfboard pin, F.Cu at (175.9, 106.5)
- added PB92: perfboard_pin, bjarkarbody:perfboard pin, F.Cu at (175.9, 109.1)
- added PB93: perfboard_pin, bjarkarbody:perfboard pin, F.Cu at (175.9, 111.6)
- added PB94: perfboard_pin, bjarkarbody:perfboard pin, F.Cu at (175.9, 114.1)
- added PB95: perfboard_pin, bjarkarbody:perfboard pin, F.Cu at (175.9, 116.7)
- added PB96: perfboard_pin, bjarkarbody:perfboard pin, F.Cu at (175.9, 119.2)
- added PB97: perfboard_pin, bjarkarbody:perfboard pin, F.Cu at (178.4, 91.3)
- added PB98: perfboard_pin, bjarkarbody:perfboard pin, F.Cu at (178.4, 93.8)
- added PB99: perfboard_pin, bjarkarbody:perfboard pin, F.Cu at (178.4, 96.4)
- J3: value Conn_01x08_Socket -> GK3_socket; footprint Connector_Wuerth:Wuerth_WR-WTB_64800811622_1x08_P1.50mm_Vertical -> bjarkarbody:gk3 connector THT
Routing:
- net DAC_BCLK: track 146.1 -> 141.4 mm, vias 9 -> 8
- net Net-(U2B--): track 29.9 -> 28.7 mm
- net GND: track 175.1 -> 174.1 mm

Commit message: silkscreen
Parts:
- added G***: LOGO, bjarkarbody:bjorktv, B.Cu at (153.1, 42.2)
Other:
- board text added: "9V TO 5V JUMPER"
- board text added: "A"
- board text added: "B"
- board text added: "BRIDGE GROUND"
- board text added: "Bradshaw Instruments Bjarkardottir 2.0"
- board text added: "D"
- board text added: "FRETBOARD"
- board text added: "G"
- board text added: "G G 5V 9V"
- board text added: "GK3"
- board text added: "HIGH E"
- board text added: "LOW E"
- board text added: "MIDI 4 MIDI 5 MIDI 2 JACK TIP JACK SLEEVE 9V GND"
- board text added: "T2 S2 T3 S3 T4 S4"

Commit message: body pcb done
Parts:
- C56: value 22uF -> 22uF 16V
- L1: footprint Inductor_SMD:L_Changjiang_FNR4020S -> Inductor_SMD:L_Sunlord_SWPA6045S
- moved L1 2.30 mm to (145.8, 130.5)
Routing:
- net Net-(D7-K): track 11.9 -> 14.9 mm
- net Net-(JP1-A): track 15.0 -> 17.7 mm
Changed lines of the file:
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@@
         (effects (font (size 1 1) (thickness 0.15)))
     )
-    (fp_text value "22uF" (at 0 1.68) (layer "F.Fab")
+    (fp_text value "22uF 16V" (at 0 1.68) (layer "F.Fab")
         (effects (font (size 1 1) (thickness 0.15)))
     )
@@
       (net 186 "unconnected-(PB45-Pin_1-Pad1)") (pinfunction "Pin_1") (pintype "no_connect"))
   )
-  (footprint "Inductor_SMD:L_Changjiang_FNR4020S" (layer "F.Cu")
-    (at 147.5 132)
-    (descr "Inductor, Changjiang, FNR4020S, 4.0x4.0x2.0mm, https://datasheet.lcsc.com/lcsc/1806131217_cjiang-Changjiang-Microelectronics-Tech-FNR5040S3R3NT_C167960.pdf")
-    (tags "Inductor wirewound power shielded")
+  (footprint "Inductor_SMD:L_Sunlord_SWPA6045S" (layer "F.Cu")
+    (at 145.75 130.5)
+    (descr "Inductor, Sunlord, SWPA6045S, 6.0x6.0x4.5mm, https://www.sunlordinc.com/UploadFiles/PDF_Cat/20120704094224784.pdf")
+    (tags "Inductor swpa")
     (property "Sheetfile" "power.kicad_sch")
     (property "Sheetname" "Power")
@@
     (property "ki_keywords" "inductor choke coil reactor magnetic")
     (attr smd)
-    (fp_text reference "L1" (at 0 -3) (layer "F.Fab")
+    (fp_text reference "L1" (at 0 -4) (layer "F.SilkS")
         (effects (font (size 1 1) (thickness 0.15)))
     )
-    (fp_text value "6.8uH" (at 0 3) (layer "F.Fab")
+    (fp_text value "6.8uH" (at 0 4) (layer "F.Fab")
         (effects (font (size 1 1) (thickness 0.15)))
     )
     (fp_text user "${REFERENCE}" (at 0 0) (layer "F.Fab")
-        (effects (font (size 0.5 0.5) (thickness 0.075)))
+        (effects (font (size 0.566667 0.566667) (thickness 0.085)))
     )
-    (fp_line (start -2.26 -2.26) (end -2.26 -2.11)
+    (fp_line (start -3.26 -3.26) (end -3.26 -3.11)
       (stroke (width 0.12) (type solid)) (layer "F.SilkS"))
-    (fp_line (start -2.26 -2.26) (end 2.26 -2.26)
+    (fp_line (start -3.26 -3.26) (end 3.26 -3.26)
       (stroke (width 0.12) (type solid)) (layer "F.SilkS"))
-    (fp_line (start -2.26 2.26) (end -2.26 2.11)
+    (fp_line (start -3.26 3.26) (end -3.26 3.11)
       (stroke (width 0.12) (type solid)) (layer "F.SilkS"))
-    (fp_line (start -2.26 2.26) (end 2.26 2.26)
+    (fp_line (start -3.26 3.26) (end 3.26 3.26)
       (stroke (width 0.12) (type solid)) (layer "F.SilkS"))
-    (fp_line (start 2.26 -2.26) (end 2.26 -2.11)
+    (fp_line (start 3.26 -3.26) (end 3.26 -3.11)
       (stroke (width 0.12) (type solid)) (layer "F.SilkS"))
-    (fp_line (start 2.26 2.26) (end 2.26 2.11)
+    (fp_line (start 3.26 3.26) (end 3.26 3.11)
       (stroke (width 0.12) (type solid)) (layer "F.SilkS"))
-    (fp_line (start -2.3 -2.25) (end -2.3 2.25)
+    (fp_line (start -3.35 -3.25) (end -3.35 3.25)
       (stroke (width 0.05) (type solid)) (layer "F.CrtYd"))
-    (fp_line (start -2.3 2.25) (end 2.3 2.25)
+    (fp_line (start -3.35 3.25) (end 3.35 3.25)
       (stroke (width 0.05) (type solid)) (layer "F.CrtYd"))
-    (fp_line (start 2.3 -2.25) (end -2.3 -2.25)
+    (fp_line (start 3.35 -3.25) (end -3.35 -3.25)
       (stroke (width 0.05) (type solid)) (layer "F.CrtYd"))
-    (fp_line (start 2.3 2.25) (end 2.3 -2.25)
+    (fp_line (start 3.35 3.25) (end 3.35 -3.25)
       (stroke (width 0.05) (type solid)) (layer "F.CrtYd"))
-    (fp_line (start -2 -2) (end -2 2)
+    (fp_line (start -3 -3) (end -3 3)
       (stroke (width 0.1) (type solid)) (layer "F.Fab"))
-    (fp_line (start -2 2) (end 2 2)
+    (fp_line (start -3 3) (end 3 3)
       (stroke (width 0.1) (type solid)) (layer "F.Fab"))
-    (fp_line (start 2 -2) (end -2 -2)
+    (fp_line (start 3 -3) (end -3 -3)
       (stroke (width 0.1) (type solid)) (layer "F.Fab"))
-    (fp_line (start 2 2) (end 2 -2)
+    (fp_line (start 3 3) (end 3 -3)
       (stroke (width 0.1) (type solid)) (layer "F.Fab"))
-    (pad "1" smd rect (at -1.5 0) (size 1.1 3.7) (layers "F.Cu" "F.Paste" "F.Mask")
+    (pad "1" smd rect (at -2.25 0) (size 1.7 5.7) (layers "F.Cu" "F.Paste" "F.Mask")
       (net 87 "Net-(D7-K)") (pinfunction "1") (pintype "passive"))
-    (pad "2" smd rect (at 1.5 0) (size 1.1 3.7) (layers "F.Cu" "F.Paste" "F.Mask")
+    (pad "2" smd rect (at 2.25 0) (size 1.7 5.7) (layers "F.Cu" "F.Paste" "F.Mask")
       (net 107 "Net-(JP1-A)") (pinfunction "2") (pintype "passive"))
-    (model "${KICAD7_3DMODEL_DIR}/Inductor_SMD.3dshapes/L_Changjiang_FNR4020S.wrl"
+    (model "${KICAD7_3DMODEL_DIR}/Inductor_SMD.3dshapes/L_Sunlord_SWPA6045S.wrl"
       (offset (xyz 0 0 0))
       (scale (xyz 1 1 1))
@@
   (segment (start 131.1 109.9) (end 134.8 109.9) (width 0.2) (layer "B.Cu") (net 84))
   (segment (start 170.78 109.02) (end 168.24 109.02) (width 0.5) (layer "F.Cu") (net 85))
-  (segment (start 146 136.5) (end 146 132) (width 0.25) (layer "F.Cu") (net 87))
+  (segment (start 145.7 132.7) (end 145.7 136.8) (width 0.5) (layer "F.Cu") (net 87))
+  (segment (start 145.7 136.8) (end 145.5 137) (width 0.5) (layer "F.Cu") (net 87))
   (segment (start 145.5 137) (end 146 136.5) (width 0.25) (layer "F.Cu") (net 87))
+  (segment (start 143.5 130.5) (end 145.7 132.7) (width 0.5) (layer "F.Cu") (net 87))
   (segment (start 141.975 135.7) (end 141.975 136.095) (width 0.25) (layer "F.Cu") (net 87))
   (segment (start 140.275 134) (end 141.975 135.7) (width 0.25) (layer "F.Cu") (net 87))
@@
   (segment (start 154.35 140.175) (end 155.5 139.025) (width 0.25) (layer "F.Cu") (net 107))
   (segment (start 155.5 139.025) (end 156 138.525) (width 0.25) (layer "F.Cu") (net 107))
-  (segment (start 153.65 136.65) (end 156 136.65) (width 0.25) (layer "F.Cu") (net 107))
   (segment (start 152.5 140.175) (end 154.35 140.175) (width 0.25) (layer "F.Cu") (net 107))
-  (segment (start 149 132) (end 153.65 136.65) (width 0.25) (layer "F.Cu") (net 107))
+  (segment (start 155.5 138) (end 155.5 139.025) (width 0.5) (layer "F.Cu") (net 107))
+  (segment (start 148 130.5) (end 155.5 138) (width 0.5) (layer "F.Cu") (net 107))
   (segment (start 156 138.525) (end 156 136.65) (width 0.25) (layer "F.Cu") (net 107))
   (segment (start 136.41 107.415) (end 136.41 110.96) (width 0.2) (layer "F.Cu") (net 108))
