File: pcb/body/power.kicad_sch (KiCad schematic)
At the start: 18 parts, among them J8 Barrel_Jack_Switch, J9 Battery_Power, U5 AP7313-18SAG, U7 TPS54331DR

Commit message: lots more layout
Parts:
- removed J8: Barrel_Jack_Switch, Connector_BarrelJack:BarrelJack_Horizontal, symbol Connector:Barrel_Jack_Switch
- added J8: 9V_POWER_INPUT, Connector_PinHeader_2.54mm:PinHeader_1x02_P2.54mm_Horizontal, symbol Connector:Conn_01x02_Pin
- renumbered C61 to C56, C62 to C57, C63 to C58, C64 to C59, C65 to C61, C66 to C63, JP7 to JP1, R43 to R46, R44 to R47, R45 to R48, U7 to U8
Connections:
- net +9V: now also J8.1 (Pin_1)
- net GND: now also J8.2 (Pin_2)
- no-connect marks 2 -> 1

Commit message: haven't committed for a bit
Parts:
- removed J8: 9V_POWER_INPUT, Connector_PinHeader_2.54mm:PinHeader_1x02_P2.54mm_Horizontal, symbol Connector:Conn_01x02_Pin
- renumbered J9 to J7

Commit message: getting there
Parts:
- U8: symbol stomp:TPS54331DR -> bjarkarbody:TPS54331DR
Changed lines of the file:
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@@
+    )
+  )
+  (symbol (lib_id "power:PWR_FLAG") (at 71.12 43.18 180) (unit 1)
+    (in_bom yes) (on_board yes) (dnp no) (fields_autoplaced)
+    (property "Reference" "#FLG02" (at 71.12 45.085 0)
+      (effects (font (size 1.27 1.27)) hide)
+    )
+    (property "Value" "PWR_FLAG" (at 71.12 47.3155 0)
+      (effects (font (size 1.27 1.27)))
+    )
+    (property "Footprint" "" (at 71.12 43.18 0)
+      (effects (font (size 1.27 1.27)) hide)
+    )
+    (property "Datasheet" "~" (at 71.12 43.18 0)
+      (effects (font (size 1.27 1.27)) hide)
+    )
+    (pin "1")
+    (instances
+      (project "body"
+        (path "/392bd065-a607-4eff-83a3-798a3e7c56fd/1a6ed37c-c9ef-40ab-9127-b7ac3319730a"
+          (reference "#FLG02") (unit 1)
+        )
+      )
     )
   )
@@
     )
   )
-  (symbol (lib_id "stomp:TPS54331DR") (at 115.57 106.68 0) (unit 1)
+  (symbol (lib_id "bjarkarbody:TPS54331DR") (at 115.57 106.68 0) (unit 1)
     (in_bom yes) (on_board yes) (dnp no) (fields_autoplaced)
     (property "Reference" "U8" (at 115.57 96.0501 0)
@@
       (effects (font (size 1.27 1.27)))
     )
-    (property "Footprint" "Package_SO:SOIC-8_3.9x4.9mm_P1.27mm" (at 116.84 115.57 0)
+    (property "Footprint" "Package_SO:SOIC-8_3.9x4.9mm_P1.27mm" (at 116.84 113.03 0)
       (effects (font (size 1.27 1.27) italic) (justify left) hide)
     )
-    (property "Datasheet" "http://www.ti.com/lit/ds/symlink/tps54331.pdf" (at 120.65 118.11 0)
+    (property "Datasheet" "http://www.ti.com/lit/ds/symlink/tps54331.pdf" (at 120.65 115.57 0)
       (effects (font (size 1.27 1.27)) hide)
     )
@@
     )
   )
+  (symbol (lib_id "power:PWR_FLAG") (at 59.69 43.18 180) (unit 1)
+    (in_bom yes) (on_board yes) (dnp no) (fields_autoplaced)
+    (property "Reference" "#FLG01" (at 59.69 45.085 0)
+      (effects (font (size 1.27 1.27)) hide)
+    )
+    (property "Value" "PWR_FLAG" (at 59.69 47.3155 0)
+      (effects (font (size 1.27 1.27)))
+    )
+    (property "Footprint" "" (at 59.69 43.18 0)
+      (effects (font (size 1.27 1.27)) hide)
+    )
+    (property "Datasheet" "~" (at 59.69 43.18 0)
+      (effects (font (size 1.27 1.27)) hide)
+    )
+    (pin "1")
+    (instances
+      (project "body"
+        (path "/392bd065-a607-4eff-83a3-798a3e7c56fd/1a6ed37c-c9ef-40ab-9127-b7ac3319730a"
+          (reference "#FLG01") (unit 1)
+        )
+      )
+    )
+  )
   (symbol (lib_id "power:+5V") (at 195.58 55.88 0) (unit 1)
     (in_bom yes) (on_board yes) (dnp no) (fields_autoplaced)
@@
     )
   )
+  (symbol (lib_id "power:+9V") (at 71.12 43.18 0) (unit 1)
+    (in_bom yes) (on_board yes) (dnp no) (fields_autoplaced)
+    (property "Reference" "#PWR015" (at 71.12 46.99 0)
+      (effects (font (size 1.27 1.27)) hide)
+    )
+    (property "Value" "+9V" (at 71.12 39.6781 0)
+      (effects (font (size 1.27 1.27)))
+    )
+    (property "Footprint" "" (at 71.12 43.18 0)
+      (effects (font (size 1.27 1.27)) hide)
+    )
+    (property "Datasheet" "" (at 71.12 43.18 0)
+      (effects (font (size 1.27 1.27)) hide)
+    )
+    (pin "1")
+    (instances
+      (project "body"
+        (path "/392bd065-a607-4eff-83a3-798a3e7c56fd/49208239-5efc-4c1f-9e9a-f65be854a588"
+          (reference "#PWR015") (unit 1)
+        )
+        (path "/392bd065-a607-4eff-83a3-798a3e7c56fd/aa0c40fb-2994-49a5-bcd0-92727450f40c"
+          (reference "#PWR029") (unit 1)
+        )
+        (path "/392bd065-a607-4eff-83a3-798a3e7c56fd/51ad2da4-249e-4e93-8132-64eb81709bf9"
+          (reference "#PWR043") (unit 1)
+        )
+        (path "/392bd065-a607-4eff-83a3-798a3e7c56fd/1a6ed37c-c9ef-40ab-9127-b7ac3319730a"
+          (reference "#PWR089") (unit 1)
+        )
+      )
+      (project "stomp_00"
+        (path "/8f4a2eb0-078b-46cb-b534-a4acd11d130e/9942492d-ba8b-45b2-b427-7fe14bedb7e0"
+          (reference "#PWR023") (unit 1)
+        )
+      )
+    )
+  )
   (symbol (lib_id "Device:C") (at 179.07 105.41 0) (unit 1)
     (in_bom yes) (on_board yes) (dnp no) (fields_autoplaced)
@@
         )
       )
+    )
+  )
+  (symbol (lib_id "power:+5V") (at 59.69 43.18 0) (unit 1)
+    (in_bom yes) (on_board yes) (dnp no) (fields_autoplaced)
+    (property "Reference" "#PWR088" (at 59.69 46.99 0)
+      (effects (font (size 1.27 1.27)) hide)
+    )
+    (property "Value" "+5V" (at 59.69 39.6781 0)
+      (effects (font (size 1.27 1.27)))
+    )
+    (property "Footprint" "" (at 59.69 43.18 0)
+      (effects (font (size 1.27 1.27)) hide)
+    )
+    (property "Datasheet" "" (at 59.69 43.18 0)
+      (effects (font (size 1.27 1.27)) hide)
+    )
+    (pin "1")
+    (instances
+      (project "body"
+        (path "/392bd065-a607-4eff-83a3-798a3e7c56fd/1a6ed37c-c9ef-40ab-9127-b7ac3319730a"
+          (reference "#PWR088") (unit 1)
+        )
+      )
+      (project "dk2_02_bottom"
+        (path "/87a59a99-d509-467e-85da-26d34072acb7/be1ddc4d-f499-4b75-b4b5-b626a320d90d"
+          (reference "#PWR049") (unit 1)
+        )
+      )
+      (project "stomp_00"
+        (path "/8f4a2eb0-078b-46cb-b534-a4acd11d130e"
+          (reference "#PWR06") (unit 1)
+        )
+        (path "/8f4a2eb0-078b-46cb-b534-a4acd11d130e/72df8ca6-692f-47f3-a8bd-ce94f6cd776a"
+          (reference "#PWR016") (unit 1)
+        )
+        (path "/8f4a2eb0-078b-46cb-b534-a4acd11d130e/9942492d-ba8b-45b2-b427-7fe14bedb7e0"
+          (reference "#PWR013") (unit 1)
+        )
+      )

Commit message: body pcb done
Parts:
- C56: value 22uF -> 22uF 16V
Changed lines of the file:
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@@
       (effects (font (size 1.27 1.27)) (justify left))
     )
-    (property "Value" "22uF" (at 90.551 115.5773 0)
+    (property "Value" "22uF 16V" (at 90.551 115.5773 0)
       (effects (font (size 1.27 1.27)) (justify left))
     )
