File: pcb/fretboard/shiftreg.kicad_sch (KiCad schematic)
At the start: 25 parts, among them J10 Conn_01x01_Pin, J11 Conn_01x01_Pin, J12 Conn_01x01_Pin, J13 Conn_01x01_Pin, J14 Conn_01x01_Pin, J15 Conn_01x01_Pin, J16 Conn_01x01_Pin, J17 Conn_01x01_Pin, J2 Conn_01x01_Pin, J3 Conn_01x01_Pin, J4 Conn_01x01_Pin, J5 Conn_01x01_Pin, J6 Conn_01x01_Pin, J7 Conn_01x01_Pin, J8 Conn_01x01_Pin, J9 Conn_01x01_Pin, U1 74HC165

Commit message: faffing with fretboard
Parts:
- removed J11, J13, J15, J17, J3, J5, J7, J9: Conn_01x01_Pin, Bjarkar:Bjarkar_fret_connection, symbol Connector:Conn_01x01_Pin
- J2: symbol Connector:Conn_01x01_Pin -> bjarkar:fret
- J3: renamed from J4; symbol Connector:Conn_01x01_Pin -> bjarkar:fret
- J4: renamed from J6; symbol Connector:Conn_01x01_Pin -> bjarkar:fret
- J5: renamed from J8; symbol Connector:Conn_01x01_Pin -> bjarkar:fret
- J6: renamed from J10; symbol Connector:Conn_01x01_Pin -> bjarkar:fret
- J7: renamed from J12; symbol Connector:Conn_01x01_Pin -> bjarkar:fret
- J8: renamed from J14; symbol Connector:Conn_01x01_Pin -> bjarkar:fret
- J9: renamed from J16; symbol Connector:Conn_01x01_Pin -> bjarkar:fret
