File: pcb/fretboard/shiftregx.kicad_sch (KiCad schematic)
At the start: 19 parts, among them J10 Conn_01x01_Pin, J11 Conn_01x01_Pin, J12 Conn_01x01_Pin, J13 Conn_01x01_Pin, J2 Conn_01x01_Pin, J3 Conn_01x01_Pin, J4 Conn_01x01_Pin, J5 Conn_01x01_Pin, J6 Conn_01x01_Pin, J7 Conn_01x01_Pin, J8 Conn_01x01_Pin, J9 Conn_01x01_Pin, U1 74HC165

Commit message: faffing with fretboard
Parts:
- removed J10, J11, J12, J13, J2, J3, J4, J5, J6, J7, J8, J9: Conn_01x01_Pin, Bjarkar:Bjarkar_fret_connection, symbol Connector:Conn_01x01_Pin
- added J10, J12, J2, J4, J6, J8: Conn_01x01_Pin, Bjarkar:Bjarkar_fret_connection, symbol bjarkar:fret
Connections:
- net at R1.2, U1.11 (D0): now also J2.1 (Pin_1)
- net at R6.2, U1.4 (D5): now also J12.1 (Pin_1)
- net at R4.2, U1.14 (D3): now also J8.1 (Pin_1)
- net at R2.2, U1.12 (D1): now also J4.1 (Pin_1)
- net at R5.2, U1.3 (D4): now also J10.1 (Pin_1)
- net at R3.2, U1.13 (D2): now also J6.1 (Pin_1)
