File: pcb/body2/audio.kicad_sch (KiCad schematic)
At the start: 16 parts, among them J3 GK3_socket, J4 AudioJack3_SwitchTR

Commit message: nicer layout
Parts:
- added J3: GK3_breakout, Connector_PinHeader_2.54mm:PinHeader_1x08_P2.54mm_Vertical, symbol Connector:Conn_01x08_Pin
- added J7: post_amp_breakout, Connector_PinHeader_2.54mm:PinHeader_1x08_P2.54mm_Vertical, symbol Connector:Conn_01x08_Pin
Connections:
- net GND: now also J3.7 (Pin_7), J3.8 (Pin_8), J7.7 (Pin_7), J7.8 (Pin_8)
- net codec1/LINE_IN_L: now also J7.6 (Pin_6)
- net codec1/LINE_IN_R: now also J7.5 (Pin_5)
- net codec2/LINE_IN_L: now also J7.4 (Pin_4)
- net codec2/LINE_IN_R: now also J7.3 (Pin_3)
- net codec3/LINE_IN_L: now also J7.2 (Pin_2)
- net codec3/LINE_IN_R: now also J7.1 (Pin_1)
- net pickuppair1/INPUT_1: now also J3.6 (Pin_6)
- net pickuppair1/INPUT_2: now also J3.5 (Pin_5)
- net pickuppair2/INPUT_1: now also J3.4 (Pin_4)
- net pickuppair2/INPUT_2: now also J3.3 (Pin_3)
- net pickuppair3/INPUT_1: now also J3.2 (Pin_2)
- net pickuppair3/INPUT_2: now also J3.1 (Pin_1)

Commit message: kicad 9
Parts:
- renumbered J3 to J4, J3 to J5, J7 to J6, J4 to J7, R9 to R10, R10 to R11, R11 to R12, R12 to R13, R3 to R6, R4 to R7, R6 to R8, R7 to R9
