File: pcb/body2/codec.kicad_sch (KiCad schematic)
At the start: 13 parts, among them U7 SGTL5000XNLA3

Commit message: kicad 9
Parts:
- renumbered C44 to C38, C45 to C39, C46 to C40, C47 to C41, C48 to C42, C49 to C43, FB2 to FB1, JP1 to JP12, JP1 to JP13, R1 to R56, R2 to R57, R61 to R58, U7 to U6

Commit message: layout
Parts:
- added J8: Conn_01x04_Socket, Connector_PinSocket_1.27mm:PinSocket_1x04_P1.27mm_Vertical, symbol Connector:Conn_01x04_Socket
Connections:
- net +3.3V: now also J8.2 (Pin_2), J8.3 (Pin_3)
- net SCL: now also J8.1 (Pin_1)
- net SDA: now also J8.4 (Pin_4)
Changed lines of the file:
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@@
+	)
+	(junction
+		(at 90.17 132.08)
+		(diameter 0)
+		(color 0 0 0 0)
 	)
 	(junction
@@
 	)
 	(junction
+		(at 82.55 118.11)
+		(diameter 0)
+		(color 0 0 0 0)
+	)
+	(junction
 		(at 91.44 109.22)
 		(diameter 0)
@@
 	)
 	(junction
+		(at 100.33 120.65)
+		(diameter 0)
+		(color 0 0 0 0)
+	)
+	(junction
 		(at 144.78 53.34)
 		(diameter 0)
@@
 	(wire
 		(pts
+			(xy 100.33 132.08) (xy 100.33 120.65)
+		)
+		(stroke
+			(width 0)
+			(type default)
+		)
+	)
+	(wire
+		(pts
 			(xy 115.57 73.66) (xy 121.92 73.66)
 		)
@@
 	(wire
 		(pts
+			(xy 82.55 118.11) (xy 82.55 132.08)
+		)
+		(stroke
+			(width 0)
+			(type default)
+		)
+	)
+	(wire
+		(pts
 			(xy 83.82 53.34) (xy 87.63 53.34)
 		)
@@
 	(wire
 		(pts
+			(xy 100.33 120.65) (xy 102.87 120.65)
+		)
+		(stroke
+			(width 0)
+			(type default)
+		)
+	)
+	(wire
+		(pts
 			(xy 154.94 53.34) (xy 154.94 68.58)
 		)
@@
 	(wire
 		(pts
-			(xy 66.04 120.65) (xy 102.87 120.65)
+			(xy 66.04 120.65) (xy 100.33 120.65)
+		)
+		(stroke
+			(width 0)
+			(type default)
+		)
+	)
+	(wire
+		(pts
+			(xy 82.55 118.11) (xy 134.62 118.11)
 		)
 		(stroke
@@
 	(wire
 		(pts
-			(xy 80.01 118.11) (xy 134.62 118.11)
+			(xy 80.01 118.11) (xy 82.55 118.11)
 		)
 		(stroke
@@
 	(wire
 		(pts
+			(xy 90.17 132.08) (xy 92.71 132.08)
+		)
+		(stroke
+			(width 0)
+			(type default)
+		)
+	)
+	(wire
+		(pts
 			(xy 87.63 60.96) (xy 87.63 73.66)
 		)
@@
 	(wire
 		(pts
+			(xy 95.25 132.08) (xy 100.33 132.08)
+		)
+		(stroke
+			(width 0)
+			(type default)
+		)
+	)
+	(wire
+		(pts
 			(xy 80.01 116.84) (xy 80.01 118.11)
 		)
@@
 	(wire
 		(pts
+			(xy 90.17 128.27) (xy 90.17 132.08)
+		)
+		(stroke
+			(width 0)
+			(type default)
+		)
+	)
+	(wire
+		(pts
 			(xy 91.44 109.22) (xy 92.71 109.22)
 		)
@@
 		(pts
 			(xy 125.73 92.71) (xy 134.62 92.71)
+		)
+		(stroke
+			(width 0)
+			(type default)
+		)
+	)
+	(wire
+		(pts
+			(xy 82.55 132.08) (xy 87.63 132.08)
 		)
 		(stroke
@@
 					(unit 1)
 				)
+			)
+		)
+	)
+	(symbol
+		(lib_id "power:+3.3V")
+		(at 90.17 128.27 0)
+		(unit 1)
+		(exclude_from_sim no)
+		(in_bom yes)
+		(on_board yes)
+		(dnp no)
+		(fields_autoplaced yes)
+		(property "Reference" "#PWR096"
+			(at 90.17 132.08 0)
+			(effects
+				(font
+					(size 1.27 1.27)
+				)
+				(hide yes)
+			)
+		)
+		(property "Value" "+3.3V"
+			(at 90.17 124.7681 0)
+			(effects
+				(font
+					(size 1.27 1.27)
+				)
+			)
+		)
+		(property "Footprint" ""
+			(at 90.17 128.27 0)
+			(effects
+				(font
+					(size 1.27 1.27)
+				)
+				(hide yes)
+			)
+		)
+		(property "Datasheet" ""
+			(at 90.17 128.27 0)
+			(effects
+				(font
+					(size 1.27 1.27)
+				)
+				(hide yes)
+			)
+		)
+		(property "Description" ""
+			(at 90.17 128.27 0)
+			(effects
+				(font
+					(size 1.27 1.27)
+				)
+			)
+		)
+		(pin "1"
+		)
+		(instances
+			(project "body2"
+				(path "/392bd065-a607-4eff-83a3-798a3e7c56fd/073c7d27-a0d4-435d-bbdf-4ca13a422348/c1feb4ca-8cfd-464c-87f4-c6f44369e3ef"
+					(reference "#PWR097")
+					(unit 1)
+				)
+				(path "/392bd065-a607-4eff-83a3-798a3e7c56fd/073c7d27-a0d4-435d-bbdf-4ca13a422348/c479731f-e64e-44fe-b03b-b9b0a66ef5c3"
+					(reference "#PWR096")
+					(unit 1)
+				)
+				(path "/392bd065-a607-4eff-83a3-798a3e7c56fd/073c7d27-a0d4-435d-bbdf-4ca13a422348/ef2a7711-a7c2-4878-bf74-326e38fd0dd7"
+					(reference "#PWR098")
+					(unit 1)
+				)
+			)
+		)
+	)
+	(symbol
+		(lib_id "Connector:Conn_01x04_Socket")
+		(at 92.71 137.16 270)
+		(unit 1)
+		(exclude_from_sim no)
+		(in_bom yes)
+		(on_board yes)
+		(dnp no)
+		(fields_autoplaced yes)
+		(property "Reference" "J8"
+			(at 91.44 138.8293 90)
+			(effects
+				(font
+					(size 1.27 1.27)
+				)
+			)
+		)
+		(property "Value" "Conn_01x04_Socket"
+			(at 91.44 141.2536 90)
+			(effects
+				(font
+					(size 1.27 1.27)
+				)
+			)
+		)
+		(property "Footprint" "Connector_PinSocket_1.27mm:PinSocket_1x04_P1.27mm_Vertical"
+			(at 92.71 137.16 0)
+			(effects
+				(font
+					(size 1.27 1.27)
+				)
+				(hide yes)
+			)
+		)
+		(property "Datasheet" "~"
+			(at 92.71 137.16 0)
+			(effects
+				(font
+					(size 1.27 1.27)
+				)
+				(hide yes)
+			)
+		)
+		(property "Description" "Generic connector, single row, 01x04, script generated"
+			(at 92.71 137.16 0)
+			(effects
+				(font
+					(size 1.27 1.27)
+				)
+				(hide yes)
+			)
+		)
+		(pin "4"
+		)
+		(pin "1"
+		)
+		(pin "2"
+		)
+		(pin "3"
+		)
+		(instances
+			(project ""
+				(path "/392bd065-a607-4eff-83a3-798a3e7c56fd/073c7d27-a0d4-435d-bbdf-4ca13a422348/c1feb4ca-8cfd-464c-87f4-c6f44369e3ef"
+					(reference "J9")
+					(unit 1)
+				)
+				(path "/392bd065-a607-4eff-83a3-798a3e7c56fd/073c7d27-a0d4-435d-bbdf-4ca13a422348/c479731f-e64e-44fe-b03b-b9b0a66ef5c3"
+					(reference "J8")
+					(unit 1)
+				)
+				(path "/392bd065-a607-4eff-83a3-798a3e7c56fd/073c7d27-a0d4-435d-bbdf-4ca13a422348/ef2a7711-a7c2-4878-bf74-326e38fd0dd7"
+					(reference "J10")
+					(unit 1)
+				)
