File: pcb/body2/pickuppair.kicad_sch (KiCad schematic)
At the start: 31 parts, among them U4 TL072, U5 TL072

Commit message: kicad 9
Parts:
- renumbered C21 to C10, C22 to C11, C23 to C12, C24 to C13, C25 to C14, C26 to C15, C16 to C5, C17 to C6, C18 to C7, C19 to C8, C20 to C9, D3 to D1, D4 to D2, R28 to R14, R29 to R15, R30 to R16, R31 to R17, R32 to R18, R33 to R19, R34 to R20, R35 to R21, R40 to R26, R41 to R27, U5 to U3, U4 to U3
