File: pcb/body2/body2.kicad_pcb (KiCad board)
At the start: 4 copper layers, 90 x 95 mm, 184 parts, among them J1 FRETBOARD_CONNECTION, J10 Conn_01x04_Socket, J2 Conn_02x12_Odd_Even, J3 Conn_01x10, J4 GK3_breakout, J5 GK3_socket, J6 post_amp_breakout, J7 AudioJack3_SwitchTR, J8 Conn_01x04_Socket, J9 Conn_01x04_Socket, U1 Teensy4.1, U10 AP7313-18SAG, U2 TCA9548APWR, U3 TL072, U4 TL072, U5 TL072, U6 SGTL5000XNLA3, U7 SGTL5000XNLA3, U8 SGTL5000XNLA3, U9 TPS54331DR

Commit message: pcb 2 done
Other:
- board text added: "JLCJLCJLCJLC"
Changed lines of the file:
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@@
 			)
 		)
-		(property "LCSC" "C21190"
+		(property "LCSC" "C4190"
 			(at 0 0 90)
 			(layer "F.Fab")
@@
 			)
 		)
-		(property "LCSC" "C21190"
+		(property "LCSC" "C4190"
 			(at 0 0 90)
 			(layer "F.Fab")
@@
 			)
 		)
-		(property "LCSC" "C21190"
+		(property "LCSC" "C4190"
 			(at 0 0 90)
 			(layer "F.Fab")
@@
 			)
 		)
-		(property "LCSC" "C21190"
+		(property "LCSC" "C4190"
 			(at 0 0 90)
 			(layer "F.Fab")
@@
 			)
 		)
+		(property "LCSC" "C23184"
+			(at 0 0 0)
+			(layer "F.SilkS")
+			(hide yes)
+			(effects
+				(font
+					(size 1.27 1.27)
+					(thickness 0.15)
+				)
+			)
+		)
 		(property ki_fp_filters "R_*")
 		(sheetname "/Power/")
@@
 			)
 		)
-		(property "LCSC" "C21190"
+		(property "LCSC" "C4190"
 			(at 0 0 90)
 			(layer "F.Fab")
@@
 			)
 		)
-		(property "LCSC" "C21190"
+		(property "LCSC" "C4190"
 			(at 0 0 90)
 			(layer "F.Fab")
@@
 			)
 		)
+		(property "LCSC" "C130026"
+			(at 0 0 0)
+			(layer "F.SilkS")
+			(hide yes)
+			(effects
+				(font
+					(size 1.27 1.27)
+					(thickness 0.15)
+				)
+			)
+		)
 		(property ki_fp_filters "TSSOP*4.4x7.8mm*P0.65mm*")
 		(sheetname "/")
@@
 			)
 		)
-		(property "LCSC" "C21190"
+		(property "LCSC" "C4190"
 			(at 0 0 90)
 			(layer "F.Fab")
@@
 			)
 		)
+		(property "LCSC" "C4177"
+			(at 0 0 0)
+			(layer "F.SilkS")
+			(hide yes)
+			(effects
+				(font
+					(size 1.27 1.27)
+					(thickness 0.15)
+				)
+			)
+		)
 		(property ki_fp_filters "R_*")
 		(sheetname "/Power/")
@@
 			)
 		)
-		(property "LCSC" "C21190"
+		(property "LCSC" "C4190"
 			(at 0 0 90)
 			(layer "F.Fab")
@@
 			)
 		)
-		(property "LCSC" "C21190"
+		(property "LCSC" "C4190"
 			(at 0 0 90)
 			(layer "F.Fab")
@@
 		(layer "F.SilkS")
 		(effects
+			(font
+				(size 1 1)
+				(thickness 0.1)
+			)
+			(justify left bottom)
+		)
+	)
+	(gr_text "JLCJLCJLCJLC"
+		(at 169.4 52.4 0)
+		(layer "F.SilkS")
+		(effects
